File: pcb/ioh.sch (EAGLE design)
At the start: 23 parts, among them Q1 MOSFET-NCHANNEL2N7000, Q2 MOSFET-NCHANNEL2N7000, Q3 MOSFET-NCHANNEL2N7000, Q4 MOSFET-NCHANNEL2N7000

Commit message: actually connect things
Connections:
- removed net N$15: JP2.2, U$1.CTS0
- removed net N$17: JP2.4, U$1.RX0
- removed net N$20: JP2.7, U$1.AD4
- removed net N$21: JP2.8, U$1.AD3
- removed net N$6: JP1.3, U$1.RX1
- net RXBACK: now also JP2.4, U$1.RX0
- net RXFRONT: now also JP1.3, U$1.RX1
- net TXBACK: now also JP2.7, U$1.AD4
- net TXFRONT: now also JP2.8, U$1.AD3
- net VIBE: now also JP2.2, U$1.CTS0
Changed lines of the file:
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@@
-</segment>
-</net>
-<net name="N$6" class="0">
-<segment>
-<pinref part="JP1" gate="G$1" pin="3"/>
-<pinref part="U$1" gate="G$1" pin="RX1"/>
-<wire x1="17.78" y1="78.74" x2="27.94" y2="78.74" width="0.1524" layer="91"/>
 </segment>
 </net>
@@
 </segment>
 </net>
-<net name="N$15" class="0">
-<segment>
-<pinref part="U$1" gate="G$1" pin="CTS0"/>
-<pinref part="JP2" gate="G$1" pin="2"/>
-<wire x1="68.58" y1="63.5" x2="81.28" y2="63.5" width="0.1524" layer="91"/>
-</segment>
-</net>
 <net name="N$16" class="0">
 <segment>
@@
 </segment>
 </net>
-<net name="N$17" class="0">
-<segment>
-<pinref part="U$1" gate="G$1" pin="RX0"/>
-<pinref part="JP2" gate="G$1" pin="4"/>
-<wire x1="68.58" y1="68.58" x2="81.28" y2="68.58" width="0.1524" layer="91"/>
-</segment>
-</net>
 <net name="N$18" class="0">
 <segment>
@@
 <pinref part="JP2" gate="G$1" pin="6"/>
 <wire x1="68.58" y1="73.66" x2="81.28" y2="73.66" width="0.1524" layer="91"/>
-</segment>
-</net>
-<net name="N$20" class="0">
-<segment>
-<pinref part="U$1" gate="G$1" pin="AD4"/>
-<pinref part="JP2" gate="G$1" pin="7"/>
-<wire x1="68.58" y1="76.2" x2="81.28" y2="76.2" width="0.1524" layer="91"/>
-</segment>
-</net>
-<net name="N$21" class="0">
-<segment>
-<pinref part="U$1" gate="G$1" pin="AD3"/>
-<pinref part="JP2" gate="G$1" pin="8"/>
-<wire x1="68.58" y1="78.74" x2="81.28" y2="78.74" width="0.1524" layer="91"/>
 </segment>
 </net>
@@
 <label x="-53.34" y="157.48" size="1.778" layer="95"/>
 </segment>
+<segment>
+<pinref part="U$1" gate="G$1" pin="AD4"/>
+<pinref part="JP2" gate="G$1" pin="7"/>
+<wire x1="68.58" y1="76.2" x2="81.28" y2="76.2" width="0.1524" layer="91"/>
+<label x="68.58" y="76.2" size="1.778" layer="95"/>
+</segment>
 </net>
 <net name="N$24" class="0">
@@
 <wire x1="-104.14" y1="157.48" x2="-119.38" y2="157.48" width="0.1524" layer="91"/>
 <label x="-119.38" y="157.48" size="1.778" layer="95"/>
+</segment>
+<segment>
+<pinref part="U$1" gate="G$1" pin="AD3"/>
+<pinref part="JP2" gate="G$1" pin="8"/>
+<wire x1="68.58" y1="78.74" x2="81.28" y2="78.74" width="0.1524" layer="91"/>
+<label x="68.58" y="78.74" size="1.778" layer="95"/>
 </segment>
 </net>
@@
 <label x="-111.76" y="99.06" size="1.778" layer="95"/>
 </segment>
+<segment>
+<pinref part="JP1" gate="G$1" pin="3"/>
+<pinref part="U$1" gate="G$1" pin="RX1"/>
+<wire x1="17.78" y1="78.74" x2="27.94" y2="78.74" width="0.1524" layer="91"/>
+<label x="17.78" y="78.74" size="1.778" layer="95"/>
+</segment>
 </net>
 <net name="RXBACK" class="0">
@@
 <label x="-76.2" y="99.06" size="1.778" layer="95"/>
 </segment>
+<segment>
+<pinref part="U$1" gate="G$1" pin="RX0"/>
+<pinref part="JP2" gate="G$1" pin="4"/>
+<wire x1="68.58" y1="68.58" x2="81.28" y2="68.58" width="0.1524" layer="91"/>
+<label x="68.58" y="68.58" size="1.778" layer="95"/>
+</segment>
 </net>
 <net name="N$13" class="0">
@@
 <label x="-10.16" y="162.56" size="1.778" layer="95"/>
 </segment>
-</net>
+<segment>
+<pinref part="U$1" gate="G$1" pin="CTS0"/>
+<pinref part="JP2" gate="G$1" pin="2"/>
+<wire x1="68.58" y1="63.5" x2="81.28" y2="63.5" width="0.1524" layer="91"/>
+<label x="68.58" y="63.5" size="1.778" layer="95"/>
+</segment>
+</net>

Commit message: some names
Parts:
- renumbered D1 to IRFRONT, D2 to IRBACK, JP3 to BZZ
Other:
- note added: "TODO FTDI TEST POINTS"
- note removed: "TODO BUTTON FTDI"
Changed lines of the file:
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@@
 <part name="SUPPLY5" library="SparkFun-Aesthetics" deviceset="VCC" device=""/>
 <part name="R1" library="SparkFun-Resistors" deviceset="RESISTOR" device="PTH-1/4W" value="20k"/>
-<part name="D1" library="SparkFun-LED" deviceset="LTE-302" device=""/>
+<part name="IRFRONT" library="SparkFun-LED" deviceset="LTE-302" device=""/>
 <part name="SUPPLY6" library="SparkFun-Aesthetics" deviceset="VCC" device=""/>
 <part name="R2" library="SparkFun-Resistors" deviceset="RESISTOR" device="PTH-1/4W" value="20k"/>
 <part name="Q2" library="SparkFun-DiscreteSemi" deviceset="MOSFET-NCHANNEL" device="2N7000"/>
 <part name="GND5" library="SparkFun-Aesthetics" deviceset="GND" device=""/>
-<part name="D2" library="SparkFun-LED" deviceset="LTE-302" device=""/>
+<part name="IRBACK" library="SparkFun-LED" deviceset="LTE-302" device=""/>
 <part name="SUPPLY7" library="SparkFun-Aesthetics" deviceset="VCC" device=""/>
 <part name="R3" library="SparkFun-Resistors" deviceset="RESISTOR" device="PTH-1/4W" value="20k"/>
@@
 <part name="SUPPLY9" library="SparkFun-Aesthetics" deviceset="VCCIO" device=""/>
 <part name="C1" library="SparkFun-Capacitors" deviceset="10UF-25V-20%(PTH)" device="KIT" value="10uF"/>
-<part name="JP3" library="SparkFun-Connectors" deviceset="M02" device="PTH"/>
+<part name="BZZ" library="SparkFun-Connectors" deviceset="M02" device="PTH"/>
 <part name="SUPPLY10" library="SparkFun-Aesthetics" deviceset="VCC" device=""/>
 <part name="GND9" library="SparkFun-Aesthetics" deviceset="GND" device=""/>
@@
 <plain>
 <text x="-132.08" y="180.34" size="1.778" layer="91">TODO
- BUTTON
- FTDI</text>
+ FTDI
+ TEST POINTS</text>
 </plain>
 <instances>
@@
 <instance part="SUPPLY5" gate="G$1" x="-38.1" y="106.68"/>
 <instance part="R1" gate="G$1" x="-38.1" y="99.06" rot="R90"/>
-<instance part="D1" gate="G$1" x="-96.52" y="172.72"/>
+<instance part="IRFRONT" gate="G$1" x="-96.52" y="172.72"/>
 <instance part="SUPPLY6" gate="G$1" x="-96.52" y="193.04"/>
 <instance part="R2" gate="G$1" x="-96.52" y="185.42" rot="R90"/>
 <instance part="Q2" gate="G$1" x="-96.52" y="157.48"/>
 <instance part="GND5" gate="1" x="-96.52" y="144.78"/>
-<instance part="D2" gate="G$1" x="-30.48" y="172.72"/>
+<instance part="IRBACK" gate="G$1" x="-30.48" y="172.72"/>
 <instance part="SUPPLY7" gate="G$1" x="-30.48" y="193.04"/>
 <instance part="R3" gate="G$1" x="-30.48" y="185.42" rot="R90"/>
@@
 <instance part="SUPPLY9" gate="G$1" x="-99.06" y="114.3"/>
 <instance part="C1" gate="G$1" x="139.7" y="53.34"/>
-<instance part="JP3" gate="G$1" x="30.48" y="175.26" rot="R180"/>
+<instance part="BZZ" gate="G$1" x="30.48" y="175.26" rot="R180"/>
 <instance part="SUPPLY10" gate="G$1" x="15.24" y="190.5"/>
 <instance part="GND9" gate="1" x="15.24" y="152.4"/>
@@
 </segment>
 <segment>
-<pinref part="JP3" gate="G$1" pin="1"/>
+<pinref part="BZZ" gate="G$1" pin="1"/>
 <wire x1="22.86" y1="175.26" x2="15.24" y2="175.26" width="0.1524" layer="91"/>
 <pinref part="SUPPLY10" gate="G$1" pin="VCC"/>
@@
 <segment>
 <pinref part="R2" gate="G$1" pin="1"/>
-<pinref part="D1" gate="G$1" pin="A"/>
+<pinref part="IRFRONT" gate="G$1" pin="A"/>
 <wire x1="-96.52" y1="180.34" x2="-96.52" y2="175.26" width="0.1524" layer="91"/>
 </segment>
@@
 <net name="N$11" class="0">
 <segment>
-<pinref part="D1" gate="G$1" pin="C"/>
+<pinref part="IRFRONT" gate="G$1" pin="C"/>
 <pinref part="Q2" gate="G$1" pin="D"/>
 <wire x1="-96.52" y1="167.64" x2="-96.52" y2="162.56" width="0.1524" layer="91"/>
@@
 <segment>
 <pinref part="R3" gate="G$1" pin="1"/>
-<pinref part="D2" gate="G$1" pin="A"/>
+<pinref part="IRBACK" gate="G$1" pin="A"/>
 <wire x1="-30.48" y1="180.34" x2="-30.48" y2="175.26" width="0.1524" layer="91"/>
 </segment>
@@
 <net name="N$25" class="0">
 <segment>
-<pinref part="D2" gate="G$1" pin="C"/>
+<pinref part="IRBACK" gate="G$1" pin="C"/>
 <pinref part="Q3" gate="G$1" pin="D"/>
 <wire x1="-30.48" y1="167.64" x2="-30.48" y2="162.56" width="0.1524" layer="91"/>
@@
 <segment>
 <pinref part="Q4" gate="G$1" pin="D"/>
-<pinref part="JP3" gate="G$1" pin="2"/>
+<pinref part="BZZ" gate="G$1" pin="2"/>
 <wire x1="15.24" y1="167.64" x2="15.24" y2="172.72" width="0.1524" layer="91"/>
 <wire x1="15.24" y1="172.72" x2="22.86" y2="172.72" width="0.1524" layer="91"/>

Commit message: power test points
Parts:
- added GND, VCC, VCCIO: M01PTH, SparkFun-Connectors:M01PTH
Connections:
- net GND: now also GND.1
- net VCC: now also VCC.1
- net VCCIO: now also VCCIO.1
Changed lines of the file:
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@@
 <part name="S1" library="adafruit" deviceset="40-XX" device=""/>
 <part name="GND10" library="SparkFun-Aesthetics" deviceset="GND" device=""/>
+<part name="VCC" library="SparkFun-Connectors" deviceset="M01" device="PTH"/>
+<part name="VCCIO" library="SparkFun-Connectors" deviceset="M01" device="PTH"/>
+<part name="GND" library="SparkFun-Connectors" deviceset="M01" device="PTH"/>
 </parts>
 <sheets>
@@
 <instance part="S1" gate="1" x="-114.3" y="63.5"/>
 <instance part="GND10" gate="1" x="-114.3" y="45.72"/>
+<instance part="VCC" gate="G$1" x="154.94" y="76.2" rot="R180"/>
+<instance part="VCCIO" gate="G$1" x="154.94" y="60.96" rot="R180"/>
+<instance part="GND" gate="G$1" x="154.94" y="45.72" rot="R180"/>
 </instances>
 <busses>
@@
 <wire x1="139.7" y1="45.72" x2="124.46" y2="45.72" width="0.1524" layer="91"/>
 <junction x="124.46" y="45.72"/>
+<pinref part="GND" gate="G$1" pin="1"/>
+<wire x1="147.32" y1="45.72" x2="139.7" y2="45.72" width="0.1524" layer="91"/>
+<junction x="139.7" y="45.72"/>
 </segment>
 <segment>
@@
 <wire x1="139.7" y1="55.88" x2="139.7" y2="60.96" width="0.1524" layer="91"/>
 <wire x1="139.7" y1="60.96" x2="124.46" y2="60.96" width="0.1524" layer="91"/>
+<pinref part="VCCIO" gate="G$1" pin="1"/>
+<wire x1="147.32" y1="60.96" x2="139.7" y2="60.96" width="0.1524" layer="91"/>
+<junction x="139.7" y="60.96"/>
 </segment>
 <segment>
@@
 <pinref part="SUPPLY2" gate="G$1" pin="VCC"/>
 <pinref part="BAT2" gate="G$1" pin="+"/>
-<wire x1="124.46" y1="78.74" x2="124.46" y2="73.66" width="0.1524" layer="91"/>
-</segment>
-<segment>
+<wire x1="124.46" y1="78.74" x2="124.46" y2="76.2" width="0.1524" layer="91"/>
+<pinref part="VCC" gate="G$1" pin="1"/>
+<wire x1="124.46" y1="76.2" x2="124.46" y2="73.66" width="0.1524" layer="91"/>
+<wire x1="147.32" y1="76.2" x2="124.46" y2="76.2" width="0.1524" layer="91"/>
+<junction x="124.46" y="76.2"/>
+</segment>
+<segment>

Commit message: OSH
Parts:
- added LOGO1: OSHW-LOGOS, SparkFun-Aesthetics:OSHW-LOGOS
Changed lines of the file:
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@@
 <part name="VCCIO" library="SparkFun-Connectors" deviceset="M01" device="PTH"/>
 <part name="GND" library="SparkFun-Connectors" deviceset="M01" device="PTH"/>
+<part name="LOGO1" library="SparkFun-Aesthetics" deviceset="OSHW-LOGO" device="S"/>
 </parts>
 <sheets>
@@
 <instance part="VCCIO" gate="G$1" x="154.94" y="60.96" rot="R180"/>
 <instance part="GND" gate="G$1" x="154.94" y="45.72" rot="R180"/>
+<instance part="LOGO1" gate="G$1" x="-58.42" y="48.26"/>
 </instances>
 <busses>
