File: pcb/ioh.sch (EAGLE design)
At the start: 36 parts

Commit message: playing around with layouts
Parts:
- removed FRAME1: FRAME-LEDGER, SparkFun-Aesthetics:FRAME-LEDGER
Changed lines of the file:
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@@
 <part name="JP3" library="SparkFun-Connectors" deviceset="FTDI_DEVICE" device=""/>
 <part name="GND11" library="SparkFun-Aesthetics" deviceset="GND" device=""/>
-<part name="FRAME1" library="SparkFun-Aesthetics" deviceset="FRAME-LEDGER" device=""/>
 <part name="JP4" library="SparkFun-Connectors" deviceset="M03" device="LOCK"/>
 <part name="U$2" library="ioh-1" deviceset="BSIDES" device=""/>
@@
 <instance part="JP3" gate="G$1" x="114.3" y="-172.72"/>
 <instance part="GND11" gate="1" x="104.14" y="-187.96"/>
-<instance part="FRAME1" gate="G$1" x="0" y="-279.4"/>
-<instance part="FRAME1" gate="G$2" x="330.2" y="-279.4"/>
 <instance part="JP4" gate="G$1" x="322.58" y="-165.1" rot="R90"/>
 <instance part="U$2" gate="G$1" x="309.88" y="-248.92" rot="MR0"/>
